Commit message: gazebo

File: robotiq_2f_85_gripper_gazebo/urdf/robotiq_arg2f_85.xacro (robot description, xacro)
@@ -38,4 +38,9 @@
     prefix=""
     transmission_hw_interface="$(arg transmission_hw_interface)"/>
+    <link name="base_link"/>
+    <joint name="base_link-robotiq_arg2f_base_link" type="fixed">
+      <parent link="base_link" />
+      <child link="robotiq_arg2f_base_link" />
+    </joint>
   <!--
     Attach the Gazebo model to Gazebo's world frame.

File: robotiq_2f_85_gripper_visualization/urdf/robotiq_arg2f_85_macro.xacro (robot description, xacro)
@@ -180,9 +180,4 @@
     </xacro:macro>
     <!-- base link -->
-    <!-- <link name="${prefix}base_link"/>
-    <joint name="${prefix}base_link-${prefix}robotiq_arg2f_base_link" type="fixed">
-      <parent link="${prefix}base_link" />
-      <child link="${prefix}robotiq_arg2f_base_link" />
-    </joint> -->
     <link name="${prefix}robotiq_arg2f_base_link">
         <inertial>
