Commit message: remove gazebo pkg, change name of visualization to description, add gazebo specs

File: robotiq_2f_85_gripper_description/urdf/robotiq_arg2f_85.xacro (robot description, xacro)
@@ -2,5 +2,5 @@
 <robot name="robotiq_arg2f_85_model" xmlns:xacro="http://ros.org/wiki/xacro">
    <!-- import main macro -->
-  <xacro:include filename="$(find robotiq_2f_85_gripper_visualization)/urdf/robotiq_arg2f_85_macro.xacro" />
+  <xacro:include filename="$(find robotiq_2f_85_gripper_description)/urdf/robotiq_arg2f_85_macro.xacro" />
   <!-- parameters -->
   <xacro:arg name="transmission_hw_interface" default="hardware_interface/EffortJointInterface"/>

File: robotiq_2f_85_gripper_description/urdf/robotiq_arg2f_85_macro.xacro (robot description, xacro)
@@ -1,9 +1,11 @@
 <?xml version="1.0"?>
 <robot xmlns:xacro="http://ros.org/wiki/xacro">
-  <xacro:include filename="$(find robotiq_2f_85_gripper_visualization)/urdf/inc/robotiq_arg2f_85_transmissions.xacro" />
+  <xacro:include filename="$(find robotiq_2f_85_gripper_description)/urdf/inc/robotiq_arg2f_85_transmissions.xacro" />
+  <xacro:include filename="$(find robotiq_2f_85_gripper_description)/urdf/inc/robotiq_arg2f_85_gazebo.xacro" />
   <xacro:macro name="robotiq_arg2f_85" params="
     prefix transmission_hw_interface:=hardware/interface/EffortJointInterface">
     <!-- Add URDF transmission elements (for ros_control) -->
     <xacro:robotiq_arg2f_85_transmission prefix="${prefix}" hw_interface="${transmission_hw_interface}"/>
+    <xacro:robotiq_arg2f_85_gazebo prefix="${prefix}" />
     <xacro:property name="max_effort" value="100.0" />
     <xacro:property name="max_velocity" value="2.0" />
@@ -23,5 +25,5 @@
           <origin xyz="0 0 0" rpy="0 0 0" />
           <geometry>
-            <mesh filename="package://robotiq_2f_85_gripper_visualization/meshes/visual/robotiq_arg2f_85_outer_knuckle.dae" scale="0.001 0.001 0.001"/>
+            <mesh filename="package://robotiq_2f_85_gripper_description/meshes/visual/robotiq_arg2f_85_outer_knuckle.dae" scale="0.001 0.001 0.001"/>
           </geometry>
           <material name="">
@@ -32,5 +34,5 @@
           <origin xyz="0 0 0" rpy="0 0 0" />
           <geometry>
-            <mesh filename="package://robotiq_2f_85_gripper_visualization/meshes/collision/robotiq_arg2f_85_outer_knuckle.dae" scale="0.001 0.001 0.001"/>
+            <mesh filename="package://robotiq_2f_85_gripper_description/meshes/collision/robotiq_arg2f_85_outer_knuckle.dae" scale="0.001 0.001 0.001"/>
           </geometry>
         </collision>
@@ -50,5 +52,5 @@
           <origin xyz="0 0 0" rpy="0 0 0" />
           <geometry>
-            <mesh filename="package://robotiq_2f_85_gripper_visualization/meshes/visual/robotiq_arg2f_85_outer_finger.dae" scale="0.001 0.001 0.001"/>
+            <mesh filename="package://robotiq_2f_85_gripper_description/meshes/visual/robotiq_arg2f_85_outer_finger.dae" scale="0.001 0.001 0.001"/>
           </geometry>
           <material name="">
@@ -59,5 +61,5 @@
           <origin xyz="0 0 0" rpy="0 0 0" />
           <geometry>
-            <mesh filename="package://robotiq_2f_85_gripper_visualization/meshes/collision/robotiq_arg2f_85_outer_finger.dae" scale="0.001 0.001 0.001"/>
+            <mesh filename="package://robotiq_2f_85_gripper_description/meshes/collision/robotiq_arg2f_85_outer_finger.dae" scale="0.001 0.001 0.001"/>
           </geometry>
         </collision>
@@ -77,5 +79,5 @@
           <origin xyz="0 0 0" rpy="0 0 0" />
           <geometry>
-            <mesh filename="package://robotiq_2f_85_gripper_visualization/meshes/visual/robotiq_arg2f_85_inner_knuckle.dae" scale="0.001 0.001 0.001"/>
+            <mesh filename="package://robotiq_2f_85_gripper_description/meshes/visual/robotiq_arg2f_85_inner_knuckle.dae" scale="0.001 0.001 0.001"/>
           </geometry>
           <material name="">
@@ -86,5 +88,5 @@
           <origin xyz="0 0 0" rpy="0 0 0" />
           <geometry>
-            <mesh filename="package://robotiq_2f_85_gripper_visualization/meshes/collision/robotiq_arg2f_85_inner_knuckle.dae" scale="0.001 0.001 0.001"/>
+            <mesh filename="package://robotiq_2f_85_gripper_description/meshes/collision/robotiq_arg2f_85_inner_knuckle.dae" scale="0.001 0.001 0.001"/>
           </geometry>
         </collision>
@@ -104,5 +106,5 @@
           <origin xyz="0 0 0" rpy="0 0 0" />
           <geometry>
-            <mesh filename="package://robotiq_2f_85_gripper_visualization/meshes/visual/robotiq_arg2f_85_inner_finger.dae" scale="0.001 0.001 0.001"/>
+            <mesh filename="package://robotiq_2f_85_gripper_description/meshes/visual/robotiq_arg2f_85_inner_finger.dae" scale="0.001 0.001 0.001"/>
           </geometry>
           <material name="">
@@ -113,5 +115,5 @@
           <origin xyz="0 0 0" rpy="0 0 0" />
           <geometry>
-            <mesh filename="package://robotiq_2f_85_gripper_visualization/meshes/collision/robotiq_arg2f_85_inner_finger.dae" scale="0.001 0.001 0.001" />
+            <mesh filename="package://robotiq_2f_85_gripper_description/meshes/collision/robotiq_arg2f_85_inner_finger.dae" scale="0.001 0.001 0.001" />
           </geometry>
         </collision>
@@ -226,5 +228,5 @@
         <origin xyz="0 0 0" rpy="0 0 0" />
         <geometry>
-          <mesh filename="package://robotiq_2f_85_gripper_visualization/meshes/visual/robotiq_arg2f_base_link.stl" />
+          <mesh filename="package://robotiq_2f_85_gripper_description/meshes/visual/robotiq_arg2f_base_link.stl" />
         </geometry>
         <material name="">
@@ -235,5 +237,5 @@
         <origin xyz="0 0 0" rpy="0 0 0" />
         <geometry>
-          <mesh filename="package://robotiq_2f_85_gripper_visualization/meshes/collision/robotiq_arg2f_base_link.stl" />
+          <mesh filename="package://robotiq_2f_85_gripper_description/meshes/collision/robotiq_arg2f_base_link.stl" />
         </geometry>
       </collision>
