Commit message: fix urdf, rtu node bugs,

File: robotiq_2f_85_gripper_description/urdf/robotiq_arg2f_85_macro.xacro (robot description, xacro)
@@ -179,7 +179,4 @@
             <box size="0.022 0.00635 0.0375" />
           </geometry>
-          <material name="">
-            <color rgba="0.9 0.0 0.0 1" />
-          </material>
         </collision>
       </link>
